Commit message: add parent link and origin to urdf

File: urdf/ur.urdf.xacro (robot description, xacro)
@@ -10,4 +10,6 @@
    <!-- parameters -->
    <xacro:arg name="tf_prefix" default="" />
+   <xacro:arg name="parent" default="world"/>
+   <xacro:arg name="origin" default="0 0 0 0 0 0"/>
    <xacro:arg name="joint_limit_params" default="$(find ur_description)/config/$(arg ur_type)/joint_limits.yaml"/>
    <xacro:arg name="kinematics_params" default="$(find ur_description)/config/$(arg ur_type)/default_kinematics.yaml"/>
@@ -51,6 +53,10 @@
    <xacro:property name="is_sim_gazebo" value="$(arg sim_gazebo)"/>
    <xacro:property name="is_sim_ignition" value="$(arg sim_ignition)"/>
-   <!-- create link fixed to the "world" -->
-   <link name="world" />
+   <!-- Split the origin into xyz and rpy -->
+   <xacro:property name="origin_clean" value="${'$(arg origin)'.replace('&quot;', '')}" />
+   <xacro:property name="origin_xyz" value="${origin_clean.split()[0:3]}" />
+   <xacro:property name="origin_rpy" value="${origin_clean.split()[3:6]}" />
+   <!-- create link fixed to the parent (default: world) -->
+   <link name="$(arg parent)" />
    <xacro:if value="${is_sim_gazebo or is_sim_ignition}">
      <link name="ground_plane">
@@ -81,5 +87,5 @@
      name="$(arg name)"
      tf_prefix="$(arg tf_prefix)"
-     parent="world"
+     parent="$(arg parent)"
      joint_limits_parameters_file="$(arg joint_limit_params)"
      kinematics_parameters_file="$(arg kinematics_params)"
@@ -115,6 +121,6 @@
      trajectory_port="$(arg trajectory_port)"
      >
-     <origin xyz="0 0 0" rpy="0 0 0" />          <!-- position robot in the world -->
-   </xacro:ur_robot>
+     <origin xyz="${' '.join(origin_xyz)}" rpy="${' '.join(origin_rpy)}" />
+    </xacro:ur_robot>
    <xacro:if value="$(arg sim_gazebo)">
     <!-- Gazebo plugins -->
